File: Szakdolgozat_CU/Szakdolgozat_CU.kicad_pcb (KiCad board)
At the start: 4 copper layers, 0 parts

Commit message: Update PCSU PCB routing, copper pours and vias
Parts:
- added C1: 1uF, Capacitor_SMD:C_0603_1608Metric_Pad1.08x0.95mm_HandSolder, F.Cu at (77.6, 116.7)
- added C10: 100nF, Capacitor_SMD:C_0603_1608Metric_Pad1.08x0.95mm_HandSolder, F.Cu at (118.9, 171.7)
- added C11: 10uF, Capacitor_SMD:C_0805_2012Metric_Pad1.18x1.45mm_HandSolder, F.Cu at (82.5, 128.7)
- added C12: 4.7uF, Capacitor_SMD:C_0603_1608Metric_Pad1.08x0.95mm_HandSolder, F.Cu at (96.4, 96.6)
- added C13: 100nF, Capacitor_SMD:C_0603_1608Metric_Pad1.08x0.95mm_HandSolder, F.Cu at (97.3, 81.6)
- added C14: 2.2uF, Capacitor_SMD:C_0603_1608Metric_Pad1.08x0.95mm_HandSolder, F.Cu at (122.8, 96.8)
- added C15: 1uF, Capacitor_SMD:C_0603_1608Metric_Pad1.08x0.95mm_HandSolder, F.Cu at (87.1, 132.8)
- added C16: 100nF, Capacitor_SMD:C_0603_1608Metric_Pad1.08x0.95mm_HandSolder, F.Cu at (99.4, 96.6)
- added C17: 10uF, Capacitor_SMD:C_0805_2012Metric_Pad1.18x1.45mm_HandSolder, F.Cu at (97.1, 84.6)
- added C18: 100nF, Capacitor_SMD:C_0603_1608Metric_Pad1.08x0.95mm_HandSolder, F.Cu at (88.2, 40.8)
- added C19: 100nF, Capacitor_SMD:C_0603_1608Metric_Pad1.08x0.95mm_HandSolder, F.Cu at (137.9, 31.5)
- added C2: C, Capacitor_SMD:C_0603_1608Metric_Pad1.08x0.95mm_HandSolder, F.Cu at (90.2, 105.0)
- added C20: 100nF, Capacitor_SMD:C_0603_1608Metric_Pad1.08x0.95mm_HandSolder, F.Cu at (92.5, 25.8)
- added C21: 100nF, Capacitor_SMD:C_0603_1608Metric_Pad1.08x0.95mm_HandSolder, F.Cu at (92.5, 28.3)
- added C22: 100nF, Capacitor_SMD:C_0603_1608Metric_Pad1.08x0.95mm_HandSolder, F.Cu at (92.5, 30.8)
- added C23: 100nF, Capacitor_SMD:C_0603_1608Metric_Pad1.08x0.95mm_HandSolder, F.Cu at (92.5, 33.3)
- added C24: C, Capacitor_SMD:C_0603_1608Metric_Pad1.08x0.95mm_HandSolder, F.Cu at (92.5, 35.8)
- added C3: 1uF, Capacitor_SMD:C_0603_1608Metric_Pad1.08x0.95mm_HandSolder, F.Cu at (77.6, 108.7)
- added C4: 1uF, Capacitor_SMD:C_0603_1608Metric_Pad1.08x0.95mm_HandSolder, F.Cu at (88.2, 30.8)
- added C5: C, Capacitor_SMD:C_0603_1608Metric_Pad1.08x0.95mm_HandSolder, F.Cu at (100.5, 104.7)
- added C6: 100nF, Capacitor_SMD:C_0603_1608Metric_Pad1.08x0.95mm_HandSolder, F.Cu at (118.7, 42.6)
- added C7: 100nF, Capacitor_SMD:C_0603_1608Metric_Pad1.08x0.95mm_HandSolder, F.Cu at (68.2, 123.8)
- added C8: 1uF, Capacitor_SMD:C_0603_1608Metric_Pad1.08x0.95mm_HandSolder, F.Cu at (81.1, 132.7)
- added C9: 2.2uF, Capacitor_SMD:C_0603_1608Metric_Pad1.08x0.95mm_HandSolder, F.Cu at (115.8, 113.6)
- added D1: USB_IN_R, LED_SMD:LED_0603_1608Metric_Pad1.05x0.95mm_HandSolder, F.Cu at (55.3, 134.1)
- added D2: 5V_R, LED_SMD:LED_0603_1608Metric_Pad1.05x0.95mm_HandSolder, F.Cu at (93.0, 132.6)
- added D3: 3V3_R, LED_SMD:LED_0603_1608Metric_Pad1.05x0.95mm_HandSolder, F.Cu at (85.5, 114.5)
- added IC1: STM32F446VET6, STM32F446RET:QFP50P1600X1600X160-100N, F.Cu at (111.4, 101.7)
- added IC2: W25Q256JVEIQ_TR, STM32F446RET:SON127P800X600X80-9N-D, F.Cu at (111.9, 175.0)
- added IC3: TPS2117DRLR, STM32F446RET:SOTFL50P160X60-8N, F.Cu at (84.1, 131.7)
- added J1: USB_C_Receptacle_USB2.0_16P, Connector_USB:USB_C_Receptacle_GCT_USB4105-xx-A_16P_TopMnt_Horizontal, F.Cu at (54.2, 124.8)
- added J10: M2_HALL, Connector_JST:JST_XH_S4B-XH-A-1_1x04_P2.50mm_Horizontal, F.Cu at (58.2, 107.5)
- added J11: ANT1, Connector_JST:JST_XH_S4B-XH-A-1_1x04_P2.50mm_Horizontal, F.Cu at (139.5, 89.5)
- added J12: ANT2, Connector_JST:JST_XH_S12B-XH-A-1_1x12_P2.50mm_Horizontal, F.Cu at (140.1, 69.1)
- added J13: GPS, Connector_JST:JST_XH_S4B-XH-A-1_1x04_P2.50mm_Horizontal, F.Cu at (63.1, 69.1)
- added J14: IMU, Connector_JST:JST_XH_S10B-XH-A_1x10_P2.50mm_Horizontal, F.Cu at (137.9, 119.4)
- added J15: WS, Connector_JST:JST_XH_S4B-XH-A-1_1x04_P2.50mm_Horizontal, F.Cu at (79.2, 69.1)
- added J2: Conn_01x06, Connector_PinHeader_2.54mm:PinHeader_1x06_P2.54mm_Vertical, F.Cu at (65.3, 101.0)
- added J3: Micro_SD_Card_Det_Hirose_DM3AT, Connector_Card:microSD_HC_Hirose_DM3AT-SF-PEJM5, F.Cu at (96.2, 69.9)
- added J4: M1_SPI, Connector_JST:JST_XH_S4B-XH-A-1_1x04_P2.50mm_Horizontal, F.Cu at (110.5, 150.8)
- added J5: M1_CTRL, Connector_JST:JST_XH_S6B-XH-A-1_1x06_P2.50mm_Horizontal, F.Cu at (58.1, 150.6)
- added J6: BAT, Connector_JST:JST_XH_S4B-XH-A-1_1x04_P2.50mm_Horizontal, F.Cu at (94.5, 150.8)
- added J7: M1_HALL, Connector_JST:JST_XH_S4B-XH-A-1_1x04_P2.50mm_Horizontal, F.Cu at (139.4, 134.0)
- added J8: M2_SPI, Connector_JST:JST_XH_S4B-XH-A-1_1x04_P2.50mm_Horizontal, F.Cu at (78.6, 150.9)
- added J9: M2_CTRL, Connector_JST:JST_XH_S6B-XH-A-1_1x06_P2.50mm_Horizontal, F.Cu at (126.4, 150.7)
- added JP1: Jumper_2_Small_Open, Connector_PinSocket_2.54mm:PinSocket_1x02_P2.54mm_Vertical, F.Cu at (65.0, 93.2)
- added R1: 5.1k, Resistor_SMD:R_0603_1608Metric_Pad0.98x0.95mm_HandSolder, F.Cu at (61.2, 122.2)
- added R10: 47k, Resistor_SMD:R_0603_1608Metric_Pad0.98x0.95mm_HandSolder, F.Cu at (114.1, 39.8)
- added R11: 47k, Resistor_SMD:R_0603_1608Metric_Pad0.98x0.95mm_HandSolder, F.Cu at (103.6, 84.9)
- added R12: 47k, Resistor_SMD:R_0603_1608Metric_Pad0.98x0.95mm_HandSolder, F.Cu at (101.6, 84.9)
- added R13: 10k, Resistor_SMD:R_0603_1608Metric_Pad0.98x0.95mm_HandSolder, F.Cu at (105.6, 84.9)
- added R14: 47k, Resistor_SMD:R_0603_1608Metric_Pad0.98x0.95mm_HandSolder, F.Cu at (93.6, 84.9)
- added R15: 33, Resistor_SMD:R_0603_1608Metric_Pad0.98x0.95mm_HandSolder, F.Cu at (118.5, 32.3)
- added R16: 47k, Resistor_SMD:R_0603_1608Metric_Pad0.98x0.95mm_HandSolder, F.Cu at (91.6, 84.9)
- added R17: 1k, Resistor_SMD:R_0603_1608Metric_Pad0.98x0.95mm_HandSolder, F.Cu at (59.7, 134.1)
- added R18: 1k, Resistor_SMD:R_0603_1608Metric_Pad0.98x0.95mm_HandSolder, F.Cu at (93.0, 128.6)
- added R19: 1k, Resistor_SMD:R_0603_1608Metric_Pad0.98x0.95mm_HandSolder, F.Cu at (85.5, 110.4)
- added R2: 5.1k, Resistor_SMD:R_0603_1608Metric_Pad0.98x0.95mm_HandSolder, F.Cu at (61.2, 127.3)
- added R20: 10k, Resistor_SMD:R_0603_1608Metric_Pad0.98x0.95mm_HandSolder, F.Cu at (110.6, 141.6)
- added R21: 10k, Resistor_SMD:R_0603_1608Metric_Pad0.98x0.95mm_HandSolder, F.Cu at (71.4, 47.0)
- added R22: 10k, Resistor_SMD:R_0603_1608Metric_Pad0.98x0.95mm_HandSolder, F.Cu at (122.8, 29.8)
- added R23: 4.7k, Resistor_SMD:R_0603_1608Metric_Pad0.98x0.95mm_HandSolder, F.Cu at (94.5, 115.6)
- added R24: 4.7k, Resistor_SMD:R_0603_1608Metric_Pad0.98x0.95mm_HandSolder, F.Cu at (94.5, 118.1)
- added R25: 10k, Resistor_SMD:R_0603_1608Metric_Pad0.98x0.95mm_HandSolder, F.Cu at (79.1, 141.7)
- added R26: 10k, Resistor_SMD:R_0603_1608Metric_Pad0.98x0.95mm_HandSolder, F.Cu at (72.0, 42.5)
- added R27: 4.7k, Resistor_SMD:R_0603_1608Metric_Pad0.98x0.95mm_HandSolder, F.Cu at (108.6, 119.0)
- added R28: 4.7k, Resistor_SMD:R_0603_1608Metric_Pad0.98x0.95mm_HandSolder, F.Cu at (111.1, 119.0)
- added R29: 10k, Resistor_SMD:R_0603_1608Metric_Pad0.98x0.95mm_HandSolder, F.Cu at (127.4, 77.9)
- added R3: 10k, Resistor_SMD:R_0603_1608Metric_Pad0.98x0.95mm_HandSolder, F.Cu at (103.8, 172.5)
- added R30: 10k, Resistor_SMD:R_0603_1608Metric_Pad0.98x0.95mm_HandSolder, F.Cu at (131.9, 98.8)
- added R31: 4.7k, Resistor_SMD:R_0603_1608Metric_Pad0.98x0.95mm_HandSolder, F.Cu at (73.1, 79.8)
- added R32: 4.7k, Resistor_SMD:R_0603_1608Metric_Pad0.98x0.95mm_HandSolder, F.Cu at (73.1, 76.1)
- added R4: 10k, Resistor_SMD:R_0603_1608Metric_Pad0.98x0.95mm_HandSolder, F.Cu at (103.8, 175.9)
- added R5: 10k, Resistor_SMD:R_0603_1608Metric_Pad0.98x0.95mm_HandSolder, F.Cu at (114.1, 27.3)
- added R6: 20k, Resistor_SMD:R_0603_1608Metric_Pad0.98x0.95mm_HandSolder, F.Cu at (78.1, 131.2)
- added R7: 15.4k, Resistor_SMD:R_0603_1608Metric_Pad0.98x0.95mm_HandSolder, F.Cu at (78.1, 135.1)
- added R8: 10k, Resistor_SMD:R_0603_1608Metric_Pad0.98x0.95mm_HandSolder, F.Cu at (118.9, 175.5)
- added R9: 10k, Resistor_SMD:R_0603_1608Metric_Pad0.98x0.95mm_HandSolder, F.Cu at (87.1, 128.8)
- added U1: TLV75515PDBV, Package_TO_SOT_SMD:SOT-23-5, F.Cu at (78.0, 112.8)
- added U2: USBLC6-2P6, Package_TO_SOT_SMD:SOT-666, F.Cu at (64.9, 124.8)
- added Y1: ECS-80-8-30BQ-JES-TR, STM32F446RET:ECS80830BQJESTR, F.Cu at (95.5, 105.1)
Other:
- board outline added: 98 x 98 mm

Commit message: Update CU schematic and PCB
Parts:
- added C25: 1nF, Capacitor_SMD:C_0603_1608Metric_Pad1.08x0.95mm_HandSolder, F.Cu at (101.0, 113.9)
- added C26: 1nF, Capacitor_SMD:C_0603_1608Metric_Pad1.08x0.95mm_HandSolder, F.Cu at (105.2, 113.9)
- added FB1: FerriteBead, Inductor_SMD:L_0603_1608Metric_Pad1.05x0.95mm_HandSolder, F.Cu at (89.0, 110.4)
- added JP2: Jumper_2_Small_Open, Connector_PinSocket_2.54mm:PinSocket_1x02_P2.54mm_Vertical, F.Cu at (122.9, 84.2)
- added R33: 47k, Resistor_SMD:R_0603_1608Metric_Pad0.98x0.95mm_HandSolder, F.Cu at (102.1, 124.7)
- added R34: 47k, Resistor_SMD:R_0603_1608Metric_Pad0.98x0.95mm_HandSolder, F.Cu at (102.1, 122.2)
- added R35: 47k, Resistor_SMD:R_0603_1608Metric_Pad0.98x0.95mm_HandSolder, F.Cu at (107.6, 124.7)
- added R36: 47k, Resistor_SMD:R_0603_1608Metric_Pad0.98x0.95mm_HandSolder, F.Cu at (107.5, 122.1)
- added SW1: SW_Push, Button_Switch_SMD:SW_Tactile_SPST_NO_Straight_CK_PTS636Sx25SMTRLFS, F.Cu at (79.6, 89.5)
- C2, C5: value C -> 8pF
- C24: value C -> 100nF
- J4, J8: footprint Connector_JST:JST_XH_S4B-XH-A-1_1x04_P2.50mm_Horizontal -> Connector_JST:JST_XH_S5B-XH-A-1_1x05_P2.50mm_Horizontal
- J6: footprint Connector_JST:JST_XH_S4B-XH-A-1_1x04_P2.50mm_Horizontal -> Connector_JST:JST_XH_S6B-XH-A-1_1x06_P2.50mm_Horizontal
- U1: value TLV75515PDBV -> TLV75533PDBV
- moved R26 119.2 mm to (135.7, 143.2), turned to 180 degrees
- moved R22 113.9 mm to (104.9, 142.3)
- moved R21 95.3 mm to (64.1, 142.0)
- moved C19 91.2 mm to (97.2, 113.2), turned to 180 degrees
- moved C20 90.8 mm to (109.5, 114.9), turned to 90 degrees
- moved C24 78.9 mm to (103.1, 113.9), turned to -90 degrees
- moved R8 78.7 mm to (126.4, 97.1), turned to 180 degrees
- moved C10 74.7 mm to (122.6, 97.1), turned to 180 degrees
- moved C4 74.3 mm to (91.1, 105.0), turned to -90 degrees
- moved IC2 72.2 mm to (125.9, 104.1), turned to 90 degrees
- moved C6 69.1 mm to (89.0, 105.0), turned to -90 degrees
- moved R4 67.6 mm to (126.7, 112.2), turned to 90 degrees
- moved C22 67.5 mm to (114.9, 94.5), turned to 180 degrees
- moved C21 65.9 mm to (82.7, 93.4), turned to 180 degrees
- moved R3 63.4 mm to (123.4, 112.2), turned to 90 degrees
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Connections:
- C2 pad 2: /PHO0 -> /OSC_OUT
- C5 pad 2: /PH1 -> /OSC_IN
- IC1 pad 100: GND -> /3V3
- IC1 pad 12: unconnected-(IC1-PH0-OSC_IN-Pad12) -> /OSC_IN
- IC1 pad 13: unconnected-(IC1-PH1-OSC_OUT-Pad13) -> /OSC_OUT
- IC1 pad 2: /ANT2_BUSY -> unconnected-(IC1-PE3-Pad2)
- IC1 pad 23: /M1_HALL_A -> /M2_HALL_A
- IC1 pad 24: /M1_HALL_B -> /M2_HALL_B
- IC1 pad 25: unconnected-(IC1-PA2-Pad25) -> /M1_DRVOFF
- IC1 pad 26: unconnected-(IC1-PA3-Pad26) -> /~{M1_FAULT}
- IC1 pad 29: /~{M1_SCS} -> /~{M1_CS}
- IC1 pad 3: /~{ANT2_CS} -> unconnected-(IC1-PE4-Pad3)
- IC1 pad 33: /~{M2_SCS} -> /~{M1_SLEEP}
- IC1 pad 34: /BAT_V -> /M1_IPROPI
- IC1 pad 35: /M1_IPROPI -> /M2_IPROPI
- IC1 pad 36: /M2_IPROPI -> /BAT_V
- IC1 pad 37: /M1_PH/IN2 -> /~{M2_CS}
- IC1 pad 38: /M1_EN/IN1 -> unconnected-(IC1-PE7-Pad38)
- IC1 pad 39: /M1_DRVOFF -> /~{BAT_FAULT}
- IC1 pad 40: /M2_HALL_A -> /M1_PH/IN2
- IC1 pad 41: /~{M1_FAULT} -> unconnected-(IC1-PE10-Pad41)
- IC1 pad 42: /M2_HALL_B -> /M1_EN/IN1
- IC1 pad 43: /~{M1_SLEEP} -> unconnected-(IC1-PE12-Pad43)
- IC1 pad 55: /~{FLASH_CS} -> /ANT1_TX
- IC1 pad 56: /~{FLASH_WP} -> /ANT1_RX
- IC1 pad 58: /~{IMU_CS} -> /~{FLASH_WP}
- IC1 pad 59: /IMU_INT -> /~{FLASH_CS}
- IC1 pad 61: unconnected-(IC1-PD14-Pad61) -> /IMU_INT
- IC1 pad 62: unconnected-(IC1-PD15-Pad62) -> /~{IMU_CS}
- IC1 pad 63: unconnected-(IC1-PC6-Pad63) -> /M1_HALL_A
- IC1 pad 64: unconnected-(IC1-PC7-Pad64) -> /M1_HALL_B
- IC1 pad 67: /USB_USE -> unconnected-(IC1-PA8-Pad67)
- IC1 pad 68: /GPS_TX -> /ANT2_TXEN
- IC1 pad 69: /GPS_RX -> /ANT2_RXEN
- IC1 pad 7: /ANT2_DIO1 -> /~{ANT2_CS}
- IC1 pad 8: /ANT2_TXEN -> unconnected-(IC1-PC14-OSC32_IN-Pad8)
- IC1 pad 80: /SDIO_CK -> /SDIO_CLK
- IC1 pad 81: /SDIO_DET -> unconnected-(IC1-PD0-Pad81)
- IC1 pad 82: unconnected-(IC1-PD1-Pad82) -> /ANT2_DIO1
- IC1 pad 84: unconnected-(IC1-PD3-Pad84) -> /ANT2_BUSY
- IC1 pad 85: unconnected-(IC1-PD4-Pad85) -> /~{ANT2_RESET}
- IC1 pad 86: /ANT1_TX -> /GPS_TX
- IC1 pad 87: /ANT1_RX -> /GPS_RX
- IC1 pad 9: /ANT2_RXEN -> /USB_SENSE
- IC1 pad 95: unconnected-(IC1-PB-Pad95) -> /SCK
- IC1 pad 96: unconnected-(IC1-PB9-Pad96) -> /SDA
- IC1 pad 98: unconnected-(IC1-PE1-Pad98) -> /SD_DET
- IC1 pad 99: /3V3 -> GND
- IC2 pad 2: /FLASH_MISO -> /SPI2_MISO
- IC2 pad 5: /FLASH_MOSI -> /SPI2_MOSI
- IC2 pad 6: /FLASH_CLK -> /SPI2_SCK
- IC3 pad 8: /USB_USE -> /USB_SENSE
- J13 pad 4: /5V_SYSTEM -> /5V_SYS
- J14 pad 1: /5V -> /5V_SYS
- J14 pad 3: /IMU_SCLK -> /SPI2_SCK
- J14 pad 4: /IMU_MOSI -> /SPI2_MOSI
- J14 pad 7: /IMU_MISO -> /SPI2_MISO
- J4 pad 1: /M1_SCK -> GND
- J4 pad 2: /~{M1_SCS} -> /M_SCK
- J4 pad 3: /M1_SDO -> /~{M1_CS}
- J4 pad 4: /M1_SDI -> /M_MISO
- J5 pad 5: /M1_IPROPI -> /M1_IPROPI_IN
- J6 pad 2: GND -> /5V
- J6 pad 3: /~{BAT_FAULT} -> GND
- J6 pad 4: /BAT_V -> GND
- J8 pad 1: /M2_SCK -> GND
- J8 pad 2: /~{M2_SCS} -> /M_SCK
- J8 pad 3: /M2_SDO -> /~{M2_CS}
- J8 pad 4: /M2_SDI -> /M_MISO
- J9 pad 5: /M2_IPROPI -> /M2_IPROPI_IN
- R20 pad 1: /~{M1_SCS} -> /~{M1_CS}
- R22 pad 2: GND -> /3V3
- R25 pad 1: /~{M2_SCS} -> /~{M2_CS}
- R31 pad 2: /VCC -> /3V3
- R32 pad 2: /VCC -> /3V3
- R9 pad 2: /USB_USE -> /USB_SENSE
- Y1 pad 1: /PH1 -> /OSC_IN
- Y1 pad 3: /PHO0 -> /OSC_OUT
Routing:
- net /3V3: track 0.00 -> 243.6 mm, vias 0 -> 32
- net /5V_SYS: track 0.00 -> 179.7 mm, vias 0 -> 4
- net /M1_EN/IN1: track 0.00 -> 85.3 mm, vias 0 -> 1
- net /M1_PH/IN2: track 0.00 -> 83.4 mm, vias 0 -> 1
- net /M_MOSI: track 0.00 -> 82.9 mm, vias 0 -> 1
- net /M_MISO: track 0.00 -> 81.9 mm, vias 0 -> 1
- net GND: track 0.00 -> 81.4 mm, vias 0 -> 169
- net /M_SCK: track 0.00 -> 81.4 mm, vias 0 -> 1
- net /M1_DRVOFF: track 0.00 -> 73.8 mm, vias 0 -> 1
- net /~{M1_SLEEP}: track 0.00 -> 71.3 mm, vias 0 -> 1
- net /~{M1_FAULT}: track 0.00 -> 70.9 mm
- net /~{M2_SLEEP}: track 0.00 -> 66.9 mm, vias 0 -> 1
- net /~{M2_FAULT}: track 0.00 -> 64.6 mm, vias 0 -> 2
- net /ANT2_SCK: track 0.00 -> 63.2 mm, vias 0 -> 1
- net /SWDIO: track 0.00 -> 62.0 mm, vias 0 -> 1
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- added copper zone on F.Cu, net /3V3
- added copper zone on In2.Cu, net /3V3
- added copper zone on F.Cu, net /5V
- added copper zone on In2.Cu, net /5V
- added copper zone on B.Cu, net GND
- added copper zone on F.Cu, net GND
- added copper zone on In1.Cu, net GND

Commit message: CU es PCSU Rev A finished + Production Files
Parts:
- added G***: LOGO, LOGO, F.Cu at (66.0, 100.5)
- added G***: LOGO, LOGO, F.Cu at (73.9, 100.5)
- added G***: LOGO, LOGO, F.Cu at (58.9, 100.5)
- added H1_M2: MountingHole_2.2mm_M2, MountingHole:MountingHole_2.2mm_M2, F.Cu at (71.0, 87.0)
- added H2_M2: MountingHole_2.2mm_M2, MountingHole:MountingHole_2.2mm_M2, F.Cu at (127.0, 87.0)
- added H3_M2: MountingHole_2.2mm_M2, MountingHole:MountingHole_2.2mm_M2, F.Cu at (71.0, 133.0)
- added H4_M2: MountingHole_2.2mm_M2, MountingHole:MountingHole_2.2mm_M2, F.Cu at (127.0, 133.0)
- added R37: 68k, Resistor_SMD:R_0603_1608Metric_Pad0.98x0.95mm_HandSolder, F.Cu at (80.6, 125.7)
- R6: value 20k -> 47k
- R9: value 10k -> 47k
- moved R9 11.4 mm to (76.1, 125.8), turned to 0 degrees
- moved R7 11.2 mm to (88.0, 129.9), turned to 90 degrees
- moved R6 10.2 mm to (88.0, 133.9), turned to 90 degrees
- moved R24 7.99 mm to (132.4, 127.9), turned to -90 degrees
- moved C15 7.64 mm to (79.5, 133.5)
- moved C8 4.49 mm to (85.4, 133.9)
- moved R5 4.10 mm to (122.1, 85.4), turned to 180 degrees
- moved C11 4.06 mm to (78.5, 129.4)
- moved JP2 2.50 mm to (121.5, 82.1)
- moved R23 1.94 mm to (132.9, 133.5)
- moved IC3 1.55 mm to (82.5, 131.9)
Connections:
- C15 pad 2: /5V -> /USB_VBUS
- C8 pad 1: /USB_VBUS -> /5V
- IC3 pad 3: /USB_VBUS -> /5V
- IC3 pad 5: /USB_VBUS -> /5V
- IC3 pad 6: /5V -> /USB_VBUS
- IC3 pad 8: /USB_SENSE -> unconnected-(IC3-ST-Pad8)
- R6 pad 1: /USB_VBUS -> /5V
- R9 pad 1: /5V_SYS -> /USB_VBUS
Routing:
- net GND: track 81.4 -> 91.8 mm, vias 169 -> 189
- net /3V3: track 243.6 -> 249.7 mm, vias 32 -> 33
- net /USB_VBUS: track 49.4 -> 54.7 mm, vias 0 -> 2
- net /5V: track 4.12 -> 8.90 mm
- net /M1_HALL_B: track 55.8 -> 51.6 mm
- net Net-(IC3-PR1): track 7.62 -> 10.7 mm, vias 0 -> 2
- net /5V_SYS: track 179.7 -> 176.8 mm
- net /USB_SENSE: track 44.2 -> 46.6 mm
- net /BOOT0: track 33.5 -> 34.5 mm
Other:
- board text added: "Katona Attila Zoltán VZOLU7 CONTROL UNIT 2026 | REV A"
