File: Szakdolgozat_CU/Szakdolgozat_CU.kicad_sch (KiCad schematic)
At the start: 45 parts, among them IC1 STM32F446RET6TR, IC2 TPS2117DRLR, J1 USB_C_Receptacle_USB2.0_16P, J10 Conn_01x06, J11 Conn_01x04, J12 Conn_01x06, J2 Conn_01x06, J3 Conn_01x06, J4 Conn_01x04, J5 Conn_01x04, J6 Conn_01x04, J7 Conn_01x04, J8 Conn_01x04, J9 Conn_01x06, SW1 SW_Push, SW2 SW_Push, U1 TLV75515PDBV, U2 USBLC6-2P6, Y1 Crystal

Commit message: Nagyobb lábú MCU implementálás előtt
Parts:
- removed J10: Conn_01x06, Connector_PinHeader_2.54mm:PinHeader_1x06_P2.54mm_Vertical, symbol Connector_Generic:Conn_01x06
- removed J8: Conn_01x04, symbol Connector_Generic:Conn_01x04
- added C15: 4.7uF, symbol Device:C
- added C16, C18: 100nF, symbol Device:C
- added C17: 10uF, symbol Device:C
- added C19: C, symbol Device:C
- added FB1: FerriteBead, symbol Device:FerriteBead
- added IC3: W25Q256JVEIQ_TR, SON127P800X600X80-9N-D, symbol W25Q256JVEIQ_TR:W25Q256JVEIQ_TR
- added J10: Conn_01x10, Connector_PinHeader_1.00mm:PinHeader_1x10_P1.00mm_Vertical, symbol Connector_Generic:Conn_01x10
- added J13: Micro_SD_Card_Det_Hirose_DM3AT, Connector_Card:microSD_HC_Hirose_DM3AT-SF-PEJM5, symbol Connector:Micro_SD_Card_Det_Hirose_DM3AT
- added J14, J15: Conn_01x04, Connector_PinHeader_2.54mm:PinHeader_1x04_P2.54mm_Vertical, symbol Connector_Generic:Conn_01x04
- added J9: Conn_01x04, symbol Connector_Generic:Conn_01x04
- added JP1: Jumper_2_Small_Open, Connector_PinSocket_2.54mm:PinSocket_1x02_P2.54mm_Vertical, symbol Jumper:Jumper_2_Small_Open
- added R10, R11, R12, R13, R14: 47k, symbol Device:R
- added R15, R17, R18, R19, R24, R25, R26, R27, R28, R29, R30: 10k, symbol Device:R
- added R16: 33, symbol Device:R
- added R20, R21, R22, R23: 4.7k, symbol Device:R
- J8: renamed from J9; value Conn_01x06 -> Conn_01x10; symbol Connector_Generic:Conn_01x06 -> Connector_Generic:Conn_01x12
Connections:
- net 3V3: now also IC1.1 (VBAT), C15.2, C16.2, C17.2, C18.1, FB1.1, IC3.8 (VCC), J13.4 (VDD), J14.1 (Pin_1), J15.1 (Pin_1), JP1.1 (A), R10.1, R11.1, R12.1, R13.1, R14.1, R15.1, R17.1, R18.1, R19.1, R20.1, R21.1, R22.1, R23.1, R24.2, R25.2, R26.2, R27.2, R28.2, R29.2; no longer C11.2, C12.2, IC1.13 (VDDA/VREF+), J12.1 (Pin_1)
- net 5V: now also C4.2, IC2.6 (VIN2), J7.1 (Pin_1), J8.1 (Pin_1), J10.1 (Pin_1)
- net 5V_SYS: no longer C4.2, IC2.6 (VIN2)
- net GND: now also J7.2 (Pin_2), J8.12 (Pin_12), J8.2 (Pin_2), C15.1, C16.1, C17.1, C18.2, C19.2, IC3.4 (GND), IC3.9 (EP), J10.10 (Pin_10), J10.2 (Pin_2), J13.10 (DET_A), J13.6 (VSS), J13.SH (SHIELD), J14.4 (Pin_4), J15.4 (Pin_4), J9.1 (Pin_1), R30.2
- net ANT1_TX: now reaches J7.3 (Pin_3)
- net ANT1_RX: now reaches J7.4 (Pin_4)
- net ANT2_SCK: now reaches J8.3 (Pin_3)
- net ANT2_MOSI: now reaches J8.4 (Pin_4)
- net ATN2_MISO: now reaches J8.5 (Pin_5)
- net ~{ANT2_CS}: now reaches J8.6 (Pin_6)
- net ~{ANT2_CS}: now also R25.1
- net M1_PH/IN2: now reaches J2.1 (Pin_1)
- net M1_EN/IN1: now reaches J2.2 (Pin_2)
- net M1_DRVOFF: now reaches J2.3 (Pin_3)
- net ~{M1_FAULT}: now reaches J2.4 (Pin_4)
- net ~{M1_FAULT}: now also R28.1
- net M1_IPROPI: now reaches J2.5 (Pin_5)
- net ~{M1_SLEEP}: now reaches J2.6 (Pin_6)
- net M2_PH/IN2: now reaches J3.1 (Pin_1)
- net M2_EN/IN1: now reaches J3.2 (Pin_2)
- net M2_DRVOFF: now reaches J3.3 (Pin_3)
- net ~{M2_FAULT}: now reaches J3.4 (Pin_4)
- net ~{M2_FAULT}: now also R29.1
- net M2_IPROPI: now reaches J3.5 (Pin_5)
- net ~{M2_SLEEP}: now reaches J3.6 (Pin_6)
- net M1_SCK: now reaches J4.1 (Pin_1)
- net ~{M1_SCS}: now reaches J4.2 (Pin_2)
- net ~{M1_SCS}: now also R27.1
- net M1_SDO: now reaches J4.3 (Pin_3)
- net M1_SDI: now reaches J4.4 (Pin_4)
- net M2_SCK: now reaches J5.1 (Pin_1)
- net ~{M2_SCS}: now reaches J5.2 (Pin_2)
- net ~{M2_SCS}: now also R26.1
- net M2_SDO: now reaches J5.3 (Pin_3)
- net M2_SDI: now reaches J5.4 (Pin_4)
- net BATTERY_V renamed BAT_V
- net BAT_V: now also C19.1
- net BATTER_FAULT_N renamed ~{BAT_FAULT}
- net ~{BAT_FAULT}: now also R30.1
- new net: J13.5 (CLK), R16.2
- new net: J13.1 (DAT2), R14.2
- new net: J13.2 (DAT3/CD), R13.2
- new net: J13.8 (DAT1), R11.2
- new net 3V3A: C11.2, C12.2, FB1.2, IC1.13 (VDDA/VREF+)
- new net 5V_SYSTEM: J9.4 (Pin_4)
- new net ANT2_BUSY: J8.7 (Pin_7)
- new net ANT2_DIO1: J8.9 (Pin_9)
- new net ANT2_RXEN: J8.11 (Pin_11)
- new net ANT2_TXEN: J8.10 (Pin_10)
- new net FLASH_CLK: IC3.6 (CLK)
- new net FLASH_MISO: IC3.2 (DO(IO1))
- new net FLASH_MOSI: IC3.5 (DI(IO0))
- new net IMU_INT: J10.8 (Pin_8)
- new net IMU_MISO: J10.7 (Pin_7)
- new net IMU_MOSI: J10.4 (Pin_4)
- new net IMU_SCLK: J10.3 (Pin_3)
- new net M1_HALL_A: J14.2 (Pin_2), R20.2
- new net M1_HALL_B: J14.3 (Pin_3), R21.2
- new net M2_HALL_A: J15.2 (Pin_2), R22.2
- new net M2_HALL_B: J15.3 (Pin_3), R23.2
- new net RTX_GPS: J9.3 (Pin_3)
- new net SDIO_CLK: R16.1
- new net SDIO_CMD: J13.3 (CMD), R10.2
- new net SDIO_D0: J13.7 (DAT0), R12.2
- new net SD_DET: J13.9 (DET_B), R15.2
- new net TX_GPS: J9.2 (Pin_2)
- new net VTREF: J12.1 (Pin_1), JP1.2 (B)
- new net ~{ANT2_RESET}: J8.8 (Pin_8)
- new net ~{FLASH_CS}: IC3.1 (~{CS}), R17.2
- new net ~{FLASH_HOLD}: IC3.7 (IO3), R19.2
- new net ~{FLASH_WP}: IC3.3 (IO2), R18.2
- new net ~{IMU_CS}: J10.9 (Pin_9), R24.1
- no-connect marks 2 -> 4
Other:
- note added: "(analog input)"
- note added: "(analog)"
- note added: "(elv van felhuzo ellenallas a boardon, de rarakok)"
- note added: "(encoder mode)"
- note added: "(meg nincs teljesen bekötve; de nem lesz elég)"
- note added: "(nem egyertelmu h benne van e felhuzo ellenallas v erre kell)"
- note added: "(sima gnd 5V es 3V3 kivezetes)"
- note added: "1 bit connection"
- note added: "5V for MCU"
- note added: "Card in: LOW Card not in: HIGH (card close con between DET_B and DET_A)"
- note added: "Clock beallitas: https://blog.devgenius.io/mastering-the-stm32-clock-tree-flash-latency-with-cubemx-36520df301b9"
- note added: "Common pin connections:"
- note added: "Datasheet: https://www.mouser.com/datasheet/2/400/PS-MPU-9250A-01-v1.1-1313803.pdf"
- note added: "FOOTPRINTEKET KICSERELNI (KELL H A KORVANALA IS JO LEGYEN!)"
- note added: "Flash + SD card"
- note added: "Forrás: https://resources.altium.com/p/design-your-own-usb-microsd-card-reader-pcb"
- note added: "GPS:"
- note added: "I2C: all in one"
- note added: "IMU:"
- note added: "Incoming data from Motors:"
- note added: "Kesobbi fejlesztes (esetleg kovetkezo iteracio): rarakni magat az antennamodulokat a nyakra"
- note added: "LEDek meg hianyoznak!"
- note added: "MCU 2:"
- note added: "MCU-hoz: 100nF-es kapcatior a battery V-hez"
- note added: "Motor 1:"
- note added: "Motor 2:"
- note added: "Power out:"
- note added: "R16- éltompitásra; ha nem kell: 0 ohm-os oda"
- note added: "SPI1: LoRa telemetry modul SPI2: Motor1 + Motor2 SPI3: Flash + IMU"
- note added: "Wheather Station:"
- note added: "ebbe meg nem vok 100% biztos"
- note added: "in case no USB is avaliable (It can be also unsoldered...)"
- note added: "use it for USB sense (noraml GPIO can be used for it)"
- note removed: "Flash"
- moved on the sheet: J11, J12, J4, J5, J6, J7

Commit message: Schematics nagyjából kész
Parts:
- added C20: 1uF, symbol Device:C
- added C21, C25, C26, C27, C28, C29, C30: 100nF, symbol Device:C
- added C22, C23: 2.2uF, symbol Device:C
- added C24: 4.7uF, symbol Device:C
- added FB2: FerriteBead, symbol Device:FerriteBead
- added IC4: STM32F446VET6, QFP50P1600X1600X160-100N, symbol STM32F446VET:STM32F446VET6
- added R31, R32: 4.7k, symbol Device:R
- added Y2: ECS-80-8-30BQ-JES-TR, ECS80830BQJESTR, symbol ECS8083QBJ:ECS-80-8-30BQ-JES-TR
Connections:
- net 3V3: now also C24.2, C25.2, C26.1, C27.1, C28.2, C29.2, C30.2, FB2.1, IC4.11 (VDD_1), IC4.19 (VDD_2), IC4.28 (VDD_3), IC4.50 (VDD_4), IC4.6 (VBAT), IC4.75 (VDD_5), IC4.99 (VSS_5)
- net 3V3A: now also C20.2, C21.2, FB2.2, IC4.21 (VREF+), IC4.22 (VDDA)
- net 5V: now also J11.1 (Pin_1)
- net ANT1_RX: now also J7.3 (Pin_3), IC4.87 (PD6); no longer J7.4 (Pin_4)
- net ANT1_TX: now also J7.4 (Pin_4), IC4.86 (PD5); no longer J7.3 (Pin_3)
- net ANT2_BUSY: now also IC4.2 (PE3)
- net ANT2_DIO1: now also IC4.7 (PC13)
- net ANT2_MOSI: now also IC4.5 (PE6)
- net ANT2_RXEN: now also IC4.9 (PC15-OSC32_OUT)
- net ANT2_SCK: now also IC4.1 (PE2)
- net ANT2_TXEN: now also IC4.8 (PC14-OSC32_IN)
- net ATN2_MISO: now also IC4.4 (PE5)
- net BAT_V: now also IC4.34 (PC5)
- net BOOT0: now also IC4.94 (BOOT0)
- net D_USB_N: now also IC4.70 (PA11)
- net D_USB_P: now also IC4.71 (PA12)
- net D_USB_RAW_N: now also U2.3 (I/O2); no longer U2.1 (I/O1)
- net D_USB_RAW_P: now also U2.1 (I/O1); no longer U2.3 (I/O2)
- net GND: now also J11.2 (Pin_2), C20.1, C21.1, C22.1, C23.1, C24.1, C25.1, C26.2, C27.2, C28.1, C29.1, C30.1, IC4.10 (VSS_1), IC4.100 (VDD_6), IC4.20 (VSSA/VREF-), IC4.27 (VSS_2), IC4.49 (VSS_3), IC4.74 (VSS_4)
- net IMU_INT: now also IC4.59 (PD12)
- net M1_DRVOFF: now also IC4.39 (PE8)
- net M1_EN/IN1: now also IC4.38 (PE7)
- net M1_HALL_A: now also IC4.23 (PA0)
- net M1_HALL_B: now also IC4.24 (PA1)
- net M1_IPROPI: now also IC4.35 (PB0)
- net M1_PH/IN2: now also IC4.37 (PB2)
- net M2_DRVOFF: now also IC4.46 (PE15)
- net M2_EN/IN1: now also IC4.45 (PE14)
- net M2_HALL_A: now also IC4.40 (PE9)
- net M2_HALL_B: now also IC4.42 (PE11)
- net M2_IPROPI: now also IC4.36 (PB1)
- net M2_PH/IN2: now also IC4.44 (PE13)
- net NRST: now also IC4.14 (NRST)
- net SDIO_CMD: now also IC4.83 (PD2)
- net SDIO_D0: now also IC4.65 (PC8)
- net SWCLK: now also IC4.76 (PA14)
- net SWDIO: now also IC4.72 (PA13)
- net SWO: now also IC4.89 (PB3)
- net USB_USE: now also IC4.67 (PA8)
- net ~{ANT2_CS}: now also IC4.3 (PE4)
- net ~{FLASH_CS}: now also IC4.55 (PD8)
- net ~{FLASH_HOLD}: now also IC4.57 (PD10)
- net ~{FLASH_WP}: now also IC4.56 (PD9)
- net ~{IMU_CS}: now also IC4.58 (PD11)
- net ~{M1_FAULT}: now also IC4.41 (PE10)
- net ~{M1_SCS}: now also IC4.29 (PA4)
- net ~{M1_SLEEP}: now also IC4.43 (PE12)
- net ~{M2_FAULT}: now also IC4.47 (PB10)
- net ~{M2_SCS}: now also IC4.33 (PC4)
- net ~{M2_SLEEP}: now also IC4.51 (PB12)
- net SDA: now reaches J11.3 (Pin_3)
- net SDA: now also R31.1
- net SCK: now reaches J11.4 (Pin_4)
- net SCK: now also R32.1
- net SDIO_D2: now reaches J13.1 (DAT2), R14.2
- net SDIO_D2: now also IC4.78 (PC10)
- net SDIO_D3: now reaches J13.2 (DAT3/CD), R13.2
- net SDIO_D3: now also IC4.79 (PC11)
- net SDIO_D1: now reaches J13.8 (DAT1), R11.2
- net SDIO_D1: now also IC4.66 (PC9)
- net RTX_GPS renamed GPS_TX
- net GPS_TX: now also IC4.68 (PA9)
- net TX_GPS renamed GPS_RX
- net GPS_RX: now also IC4.69 (PA10)
- new net: C22.2, IC4.48 (VCAP_1)
- new net: C23.2, IC4.73 (VCAP_2)
- new net M_MISO: IC4.31 (PA6)
- new net M_MOSI: IC4.32 (PA7)
- new net M_SCK: IC4.30 (PA5)
- new net SDIO_CK: IC4.80 (PC12)
- new net SDIO_DET: IC4.81 (PD0)
- new net SPI2_MISO: IC4.53 (PB14)
- new net SPI2_MOSI: IC4.54 (PB15)
- new net SPI2_SCK: IC4.52 (PB13)
- new net VCC: R31.2, R32.2
Other:
- note added: "(ezt meg lehet csinalni 1 bit-esre is)"
- note added: "ANT2_RESET meg hianyzik!!"
- note added: "ELV FEL VAN CSERELVE??"
- note added: "ESR<2ohm"
- moved on the sheet: C1, C16, C17, C18, C2, IC3, J13, R10, R11, R12, R13, R14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

Commit message: Update PCSU PCB routing, copper pours and vias
Parts:
- removed C10, C11, C14, C7, C8, C9: 100nF, symbol Device:C
- removed C12: 1uF, symbol Device:C
- removed C13, C15: 4.7uF, symbol Device:C
- removed FB1: FerriteBead, symbol Device:FerriteBead
- removed IC1: STM32F446RET6TR, QFP50P1200X1200X160-64N, symbol STM32F446RET:STM32F446RET6TR
- removed J12: Conn_01x06, Connector_PinHeader_2.54mm:PinHeader_1x06_P2.54mm_Vertical, symbol Connector_Generic:Conn_01x06
- removed R9: 10k, symbol Device:R
- removed Y1: Crystal, symbol Device:Crystal
- added C2, C5: C, symbol Device:C
- added C21: 100nF, Capacitor_SMD:C_0603_1608Metric_Pad1.08x0.95mm_HandSolder, symbol Device:C
- added J2: Conn_01x06, Connector_PinHeader_2.54mm:PinHeader_1x06_P2.54mm_Vertical, symbol Connector_Generic:Conn_01x06
- added R5: 10k, Resistor_SMD:R_0603_1608Metric_Pad0.98x0.95mm_HandSolder, symbol Device:R
- C1: footprint (none) -> Capacitor_SMD:C_0603_1608Metric_Pad1.08x0.95mm_HandSolder
- C10: renamed from C18; footprint (none) -> Capacitor_SMD:C_0603_1608Metric_Pad1.08x0.95mm_HandSolder
- C11: renamed from C6; footprint (none) -> Capacitor_SMD:C_0805_2012Metric_Pad1.18x1.45mm_HandSolder
- C12: renamed from C24; footprint (none) -> Capacitor_SMD:C_0603_1608Metric_Pad1.08x0.95mm_HandSolder
- C13: renamed from C16; footprint (none) -> Capacitor_SMD:C_0603_1608Metric_Pad1.08x0.95mm_HandSolder
- C14: renamed from C23; footprint (none) -> Capacitor_SMD:C_0603_1608Metric_Pad1.08x0.95mm_HandSolder
- C15: renamed from C4; footprint (none) -> Capacitor_SMD:C_0603_1608Metric_Pad1.08x0.95mm_HandSolder
- C16: renamed from C25; footprint (none) -> Capacitor_SMD:C_0603_1608Metric_Pad1.08x0.95mm_HandSolder
- C17: footprint (none) -> Capacitor_SMD:C_0805_2012Metric_Pad1.18x1.45mm_HandSolder
- C18: renamed from C26; footprint (none) -> Capacitor_SMD:C_0603_1608Metric_Pad1.08x0.95mm_HandSolder
- C19: renamed from C27; footprint (none) -> Capacitor_SMD:C_0603_1608Metric_Pad1.08x0.95mm_HandSolder
- C20: renamed from C28; footprint (none) -> Capacitor_SMD:C_0603_1608Metric_Pad1.08x0.95mm_HandSolder
- C22: renamed from C29; footprint (none) -> Capacitor_SMD:C_0603_1608Metric_Pad1.08x0.95mm_HandSolder
- C23: renamed from C30; footprint (none) -> Capacitor_SMD:C_0603_1608Metric_Pad1.08x0.95mm_HandSolder
- C3: renamed from C2; footprint (none) -> Capacitor_SMD:C_0603_1608Metric_Pad1.08x0.95mm_HandSolder
- C4: renamed from C20; footprint (none) -> Capacitor_SMD:C_0603_1608Metric_Pad1.08x0.95mm_HandSolder
- C6: renamed from C21; footprint (none) -> Capacitor_SMD:C_0603_1608Metric_Pad1.08x0.95mm_HandSolder
- C8: renamed from C5; footprint (none) -> Capacitor_SMD:C_0603_1608Metric_Pad1.08x0.95mm_HandSolder
- C9: renamed from C22; footprint (none) -> Capacitor_SMD:C_0603_1608Metric_Pad1.08x0.95mm_HandSolder
- D1: value LED -> USB_IN_R; footprint (none) -> LED_SMD:LED_0603_1608Metric_Pad1.05x0.95mm_HandSolder
- D2: value LED -> 5V_R; footprint (none) -> LED_SMD:LED_0603_1608Metric_Pad1.05x0.95mm_HandSolder
- D3: value LED -> 3V3_R; footprint (none) -> LED_SMD:LED_0603_1608Metric_Pad1.05x0.95mm_HandSolder
- IC1: renamed from IC4; footprint QFP50P1600X1600X160-100N -> STM32F446RET:QFP50P1600X1600X160-100N
- IC2: renamed from IC3; footprint SON127P800X600X80-9N-D -> STM32F446RET:SON127P800X600X80-9N-D
- IC3: renamed from IC2; footprint SOTFL50P160X60-8N -> STM32F446RET:SOTFL50P160X60-8N
- J10: renamed from J15; value Conn_01x04 -> M2_HALL; footprint Connector_PinHeader_2.54mm:PinHeader_1x04_P2.54mm_Vertical -> Connector_JST:JST_XH_S4B-XH-A-1_1x04_P2.50mm_Horizontal
- J11: renamed from J7; value Conn_01x04 -> ANT1; footprint (none) -> Connector_JST:JST_XH_S4B-XH-A-1_1x04_P2.50mm_Horizontal
- J12: renamed from J8; value Conn_01x10 -> ANT2; footprint Connector_PinHeader_2.54mm:PinHeader_1x06_P2.54mm_Vertical -> Connector_JST:JST_XH_S12B-XH-A-1_1x12_P2.50mm_Horizontal
- J13: renamed from J9; value Conn_01x04 -> GPS; footprint (none) -> Connector_JST:JST_XH_S4B-XH-A-1_1x04_P2.50mm_Horizontal
- J14: renamed from J10; value Conn_01x10 -> IMU; footprint Connector_PinHeader_1.00mm:PinHeader_1x10_P1.00mm_Vertical -> Connector_JST:JST_XH_S10B-XH-A_1x10_P2.50mm_Horizontal
- J15: renamed from J11; value Conn_01x04 -> WS; footprint (none) -> Connector_JST:JST_XH_S4B-XH-A-1_1x04_P2.50mm_Horizontal
- J4: value Conn_01x04 -> M1_SPI; footprint (none) -> Connector_JST:JST_XH_S4B-XH-A-1_1x04_P2.50mm_Horizontal
- J5: renamed from J2; value Conn_01x06 -> M1_CTRL; footprint Connector_PinHeader_2.54mm:PinHeader_1x06_P2.54mm_Vertical -> Connector_JST:JST_XH_S6B-XH-A-1_1x06_P2.50mm_Horizontal
- J6: value Conn_01x04 -> BAT; footprint Connector_PinHeader_2.54mm:PinHeader_1x04_P2.54mm_Vertical -> Connector_JST:JST_XH_S4B-XH-A-1_1x04_P2.50mm_Horizontal
- J7: renamed from J14; value Conn_01x04 -> M1_HALL; footprint Connector_PinHeader_2.54mm:PinHeader_1x04_P2.54mm_Vertical -> Connector_JST:JST_XH_S4B-XH-A-1_1x04_P2.50mm_Horizontal
- J8: renamed from J5; value Conn_01x04 -> M2_SPI; footprint (none) -> Connector_JST:JST_XH_S4B-XH-A-1_1x04_P2.50mm_Horizontal
- J9: renamed from J3; value Conn_01x06 -> M2_CTRL; footprint Connector_PinHeader_2.54mm:PinHeader_1x06_P2.54mm_Vertical -> Connector_JST:JST_XH_S6B-XH-A-1_1x06_P2.50mm_Horizontal
- R10, R11, R12, R31, R32: footprint (none) -> Resistor_SMD:R_0603_1608Metric_Pad0.98x0.95mm_HandSolder
- R13: renamed from R15; footprint (none) -> Resistor_SMD:R_0603_1608Metric_Pad0.98x0.95mm_HandSolder
- R14: renamed from R13; footprint (none) -> Resistor_SMD:R_0603_1608Metric_Pad0.98x0.95mm_HandSolder
- R15: renamed from R16; footprint (none) -> Resistor_SMD:R_0603_1608Metric_Pad0.98x0.95mm_HandSolder
- R16: renamed from R14; footprint (none) -> Resistor_SMD:R_0603_1608Metric_Pad0.98x0.95mm_HandSolder
- R17: renamed from R6; footprint (none) -> Resistor_SMD:R_0603_1608Metric_Pad0.98x0.95mm_HandSolder
- R18: renamed from R7; footprint (none) -> Resistor_SMD:R_0603_1608Metric_Pad0.98x0.95mm_HandSolder
- R19: renamed from R8; footprint (none) -> Resistor_SMD:R_0603_1608Metric_Pad0.98x0.95mm_HandSolder
- R20: renamed from R27; footprint (none) -> Resistor_SMD:R_0603_1608Metric_Pad0.98x0.95mm_HandSolder
- R21: renamed from R28; footprint (none) -> Resistor_SMD:R_0603_1608Metric_Pad0.98x0.95mm_HandSolder
- R22: renamed from R30; footprint (none) -> Resistor_SMD:R_0603_1608Metric_Pad0.98x0.95mm_HandSolder
- R23: renamed from R20; footprint (none) -> Resistor_SMD:R_0603_1608Metric_Pad0.98x0.95mm_HandSolder
- R24: renamed from R21; footprint (none) -> Resistor_SMD:R_0603_1608Metric_Pad0.98x0.95mm_HandSolder
- R25: renamed from R26; footprint (none) -> Resistor_SMD:R_0603_1608Metric_Pad0.98x0.95mm_HandSolder
- R26: renamed from R29; footprint (none) -> Resistor_SMD:R_0603_1608Metric_Pad0.98x0.95mm_HandSolder
- R27: renamed from R22; footprint (none) -> Resistor_SMD:R_0603_1608Metric_Pad0.98x0.95mm_HandSolder
- R28: renamed from R23; footprint (none) -> Resistor_SMD:R_0603_1608Metric_Pad0.98x0.95mm_HandSolder
- R29: renamed from R25; footprint (none) -> Resistor_SMD:R_0603_1608Metric_Pad0.98x0.95mm_HandSolder
- R3: renamed from R17; footprint (none) -> Resistor_SMD:R_0603_1608Metric_Pad0.98x0.95mm_HandSolder
- R30: renamed from R24; footprint (none) -> Resistor_SMD:R_0603_1608Metric_Pad0.98x0.95mm_HandSolder
- R4: renamed from R18; footprint (none) -> Resistor_SMD:R_0603_1608Metric_Pad0.98x0.95mm_HandSolder
- R6: renamed from R4; footprint (none) -> Resistor_SMD:R_0603_1608Metric_Pad0.98x0.95mm_HandSolder
- R7: renamed from R3; footprint (none) -> Resistor_SMD:R_0603_1608Metric_Pad0.98x0.95mm_HandSolder
- R8: renamed from R19; footprint (none) -> Resistor_SMD:R_0603_1608Metric_Pad0.98x0.95mm_HandSolder
- R9: renamed from R5; footprint (none) -> Resistor_SMD:R_0603_1608Metric_Pad0.98x0.95mm_HandSolder
- Y1: renamed from Y2; footprint ECS80830BQJESTR -> STM32F446RET:ECS80830BQJESTR
- renumbered C19 to C24, C3 to C7, FB2 to FB1, J13 to J3
Connections:
- net VCC is gone; now on net 3V3: R31.2, R32.2
- net BOOT0: now also R5.1
- net GND: now also Y1.2 (GND_1), Y1.4 (GND_2), C2.1, C21.2, C5.1, J2.3 (Pin_3), R5.2
- net NRST: now also C21.1, J2.5 (Pin_5)
- net SWCLK: now also J2.2 (Pin_2)
- net SWDIO: now also J2.4 (Pin_4)
- net SWO: now also J2.6 (Pin_6)
- net VTREF: now also J2.1 (Pin_1)
- net PH1: now reaches Y1.1 (IN/OUT)
- net PH1: now also C5.2
- net PHO0: now reaches Y1.3 (OUT/IN)
- net PHO0: now also C2.2
Other:
- note added: "EZ BIZTOSAN JÓ?"
- note added: "MCU:"
- note removed: "(meg nincs teljesen bekötve; de nem lesz elég)"
- note removed: "8MHz"
- note removed: "BOOT and NRESET"
- note removed: "ESR<1ohm"
- note removed: "MCU"
- note removed: "MCU 2:"
- note removed: "MCU power decoupeling"
- note removed: "ugyan abbol kivinni a SPI-hoz a motorhoz mint a HW-hez"
- moved on the sheet: C12, C14, C16, C18, C19, C20, C22, C23, C4, C6, C9, FB1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

Commit message: Update CU schematic and PCB
Parts:
- removed SW1: SW_Push, symbol Switch:SW_Push
- removed U1: TLV75515PDBV, Package_TO_SOT_SMD:SOT-23-5, symbol Regulator_Linear:TLV75515PDBV
- added C25, C26: 1nF, Capacitor_SMD:C_0603_1608Metric_Pad1.08x0.95mm_HandSolder, symbol Device:C
- added JP2: Jumper_2_Small_Open, Connector_PinSocket_2.54mm:PinSocket_1x02_P2.54mm_Vertical, symbol Jumper:Jumper_2_Small_Open
- added R33, R34, R35, R36: 47k, Resistor_SMD:R_0603_1608Metric_Pad0.98x0.95mm_HandSolder, symbol Device:R
- added U1: TLV75533PDBV, Package_TO_SOT_SMD:SOT-23-5, symbol Regulator_Linear:TLV75533PDBV
- C2, C5: value C -> 8pF; footprint (none) -> Capacitor_SMD:C_0603_1608Metric_Pad1.08x0.95mm_HandSolder
- C24: value C -> 100nF; footprint (none) -> Capacitor_SMD:C_0603_1608Metric_Pad1.08x0.95mm_HandSolder
- FB1: footprint (none) -> Inductor_SMD:L_0603_1608Metric_Pad1.05x0.95mm_HandSolder
- J4, J8: footprint Connector_JST:JST_XH_S4B-XH-A-1_1x04_P2.50mm_Horizontal -> Connector_JST:JST_XH_S5B-XH-A-1_1x05_P2.50mm_Horizontal; symbol Connector_Generic:Conn_01x04 -> Connector_Generic:Conn_01x05
- J6: footprint Connector_JST:JST_XH_S4B-XH-A-1_1x04_P2.50mm_Horizontal -> Connector_JST:JST_XH_S6B-XH-A-1_1x06_P2.50mm_Horizontal; symbol Connector_Generic:Conn_01x04 -> Connector_Generic:Conn_01x06
- SW1: renamed from SW2; footprint (none) -> Button_Switch_SMD:SW_Tactile_SPST_NO_Straight_CK_PTS636Sx25SMTRLFS
Connections:
- net 5V_SYSTEM is gone; now on net 5V_SYS: J13.4 (Pin_4)
- net FLASH_CLK is gone; now on net SPI2_SCK: IC2.6 (CLK)
- net FLASH_MISO is gone; now on net SPI2_MISO: IC2.2 (DO(IO1))
- net FLASH_MOSI is gone; now on net SPI2_MOSI: IC2.5 (DI(IO0))
- net IMU_MISO is gone; now on net SPI2_MISO: J14.7 (Pin_7)
- net IMU_MOSI is gone; now on net SPI2_MOSI: J14.4 (Pin_4)
- net IMU_SCLK is gone; now on net SPI2_SCK: J14.3 (Pin_3)
- net M1_SCK is gone; now on net GND: J4.1 (Pin_1)
- net M1_SDI is gone; now on net M_MISO: J4.4 (Pin_4)
- net M2_SCK is gone; now on net GND: J8.1 (Pin_1)
- net M2_SDI is gone; now on net M_MISO: J8.4 (Pin_4)
- net PH1 is gone; now on net OSC_IN: C5.2, Y1.1 (IN/OUT)
- net PHO0 is gone; now on net OSC_OUT: C2.2, Y1.3 (OUT/IN)
- net SDIO_CK is gone; now on net SDIO_CLK: IC1.80 (PC12)
- net 3V3: now also IC1.100 (VDD_6), R22.2, JP2.1 (A), U1.5 (OUT); no longer IC1.99 (VSS_5)
- net 5V: now also J6.2 (Pin_2); no longer J14.1 (Pin_1)
- net 5V_SYS: now also J14.1 (Pin_1), U1.1 (IN), U1.3 (EN)
- net ANT1_RX: now also IC1.56 (PD9); no longer IC1.87 (PD6)
- net ANT1_TX: now also IC1.55 (PD8); no longer IC1.86 (PD5)
- net ANT2_BUSY: now also IC1.84 (PD3); no longer IC1.2 (PE3)
- net ANT2_DIO1: now also IC1.82 (PD1); no longer IC1.7 (PC13)
- net ANT2_RXEN: now also IC1.69 (PA10); no longer IC1.9 (PC15-OSC32_OUT)
- net ANT2_TXEN: now also IC1.68 (PA9); no longer IC1.8 (PC14-OSC32_IN)
- net BAT_V: now also IC1.36 (PB1), J6.6 (Pin_6); no longer IC1.34 (PC5), J6.4 (Pin_4)
- net BOOT0: now also JP2.2 (B)
- net GND: now also IC1.99 (VSS_5), J6.3 (Pin_3), J6.4 (Pin_4), C25.2, C26.2, R34.1, R36.2, U1.2 (GND); no longer IC1.100 (VDD_6), J6.2 (Pin_2), R22.2
- net GPS_RX: now also IC1.87 (PD6); no longer IC1.69 (PA10)
- net GPS_TX: now also IC1.86 (PD5); no longer IC1.68 (PA9)
- net IMU_INT: now also IC1.61 (PD14); no longer IC1.59 (PD12)
- net M1_DRVOFF: now also IC1.25 (PA2); no longer IC1.39 (PE8)
- net M1_EN/IN1: now also IC1.42 (PE11); no longer IC1.38 (PE7)
- net M1_HALL_A: now also IC1.63 (PC6); no longer IC1.23 (PA0)
- net M1_HALL_B: now also IC1.64 (PC7); no longer IC1.24 (PA1)
- net M1_IPROPI: now also IC1.34 (PC5), C25.1, R33.2, R34.2; no longer IC1.35 (PB0), J5.5 (Pin_5)
- net M1_PH/IN2: now also IC1.40 (PE9); no longer IC1.37 (PB2)
- net M2_HALL_A: now also IC1.23 (PA0); no longer IC1.40 (PE9)
- net M2_HALL_B: now also IC1.24 (PA1); no longer IC1.42 (PE11)
- net M2_IPROPI: now also IC1.35 (PB0), C26.1, R35.2, R36.1; no longer IC1.36 (PB1), J9.5 (Pin_5)
- net M_MOSI: now also J4.5 (Pin_5), J8.5 (Pin_5)
- net M_SCK: now also J4.2 (Pin_2), J8.2 (Pin_2)
- net SCK: now also IC1.95 (PB)
- net SDA: now also IC1.96 (PB9)
- net SD_DET: now also IC1.98 (PE1)
- net ~{ANT2_CS}: now also IC1.7 (PC13); no longer IC1.3 (PE4)
- net ~{ANT2_RESET}: now also IC1.85 (PD4)
- net ~{BAT_FAULT}: now also IC1.39 (PE8), J6.5 (Pin_5); no longer J6.3 (Pin_3)
- net ~{FLASH_CS}: now also IC1.59 (PD12); no longer IC1.55 (PD8)
- net ~{FLASH_WP}: now also IC1.58 (PD11); no longer IC1.56 (PD9)
- net ~{IMU_CS}: now also IC1.62 (PD15); no longer IC1.58 (PD11)
- net ~{M1_FAULT}: now also IC1.26 (PA3); no longer IC1.41 (PE10)
- net ~{M1_SLEEP}: now also IC1.33 (PC4); no longer IC1.43 (PE12)
- net OSC_IN: now reaches IC1.12 (PH0-OSC_IN)
- net OSC_OUT: now reaches IC1.13 (PH1-OSC_OUT)
- net M1_SDO renamed ~{M1_CS}
- net ~{M1_CS}: now also IC1.29 (PA4), R20.1
- net M2_SDO renamed ~{M2_CS}
- net ~{M2_CS}: now also IC1.37 (PB2), R25.1
- net SDIO_DET: no longer names the net of IC1.81 (PD0)
- net USB_USE renamed USB_SENSE
- net USB_SENSE: now also IC1.9 (PC15-OSC32_OUT); no longer IC1.67 (PA8)
- removed net ~{M1_SCS}: IC1.29 (PA4), J4.2 (Pin_2), R20.1
- removed net ~{M2_SCS}: IC1.33 (PC4), J8.2 (Pin_2), R25.1
- new net M1_IPROPI_IN: J5.5 (Pin_5), R33.1
- new net M2_IPROPI_IN: J9.5 (Pin_5), R35.1
- no-connect marks 4 -> 24
Other:
- note added: "(C close to the MCU)"
- note added: "ITT 47K ELV?"
- note added: "KONDIK elhelyezeset megegyszer atnezni; C16-os jo helyen?"
- note added: "Voltage div for IPROPI (in case of error: 5.5V)"
- note removed: "2db GND + 2db 5V vezetek?? csatik nem biztos h elbirjak"
- note removed: "ANT2_RESET meg hianyzik!!"
- note removed: "ELV FEL VAN CSERELVE??"
- note removed: "EZ meg kerdes (0.1uF elegendo elv..)"
- note removed: "FOOTPRINTEKET KICSERELNI (KELL H A KORVANALA IS JO LEGYEN!)"
- note removed: "LEDek meg hianyoznak!"
- note removed: "MCU-hoz: 100nF-es kapcatior a battery V-hez"
- moved on the sheet: C2, C5, J2, J9, JP1, R26, Y1

Commit message: CU es PCSU Rev A finished + Production Files
Parts:
- added R37: 68k, Resistor_SMD:R_0603_1608Metric_Pad0.98x0.95mm_HandSolder, symbol Device:R
- R6: value 20k -> 47k
- R9: value 10k -> 47k
Connections:
- net 5V: now also C8.1, IC3.3 (VIN1), IC3.5 (MODE), R6.1; no longer C15.2, IC3.6 (VIN2)
- net 5V_SYS: no longer R9.1
- net GND: now also R37.2
- net USB_SENSE: now also R37.1; no longer IC3.8 (ST)
- net USB_VBUS: now also C15.2, IC3.6 (VIN2), R9.1; no longer C8.1, IC3.3 (VIN1), IC3.5 (MODE), R6.1
- no-connect marks 24 -> 25
Other:
- note added: "FSYNC (GND)"
- note removed: "ITT 47K ELV?"
- note removed: "use it for USB sense (noraml GPIO can be used for it)"
- moved on the sheet: R9
