File: Szakdolgozat_PCSU/Szakdolgozat_PCSU.kicad_sch (KiCad schematic)
At the start: 0 parts

Commit message: PCSU elemek keszen de BOM nem, huzalozas meg atnezesre + atnevezesre szorul, CU-bol meg nincs meg teljesen
Parts:
- added 5VLED, D1, D2, D3, D4, D6, D7, D8: LED, symbol Device:LED
- added C10, C9: 10uF, symbol Device:C
- added C11: C, symbol Device:C
- added C12: 8200pF, symbol Device:C
- added C16, C20: 10n, symbol Device:C
- added C17, C21: 100n, symbol Device:C
- added C18: 470uF, Capacitor_THT:CP_Radial_D10.0mm_P5.00mm, symbol Device:C_Polarized
- added C19: 100uF, symbol Device:C
- added C22: 470, Capacitor_THT:CP_Radial_D10.0mm_P5.00mm, symbol Device:C_Polarized
- added C4, C5, C8: 0.1uF, symbol Device:C
- added C6, C7: 22uF, symbol Device:C
- added D5: SMCJ18CA, DIONM7959X262N, symbol SMCJ18CA:SMCJ18CA
- added D_R1, D_R2, R_IT1, R_IT2, R_M1, R_M2: 0, symbol Device:R
- added F1: SF-1206HHA3000R-2, SF1206HHA3000R2, symbol SF1206HHA3000R-2:SF-1206HHA3000R-2
- added IC1, IC2: DRV8244HQDGQRQ1, SOP50P490X110-29N, symbol DRV8244HQ:DRV8244HQDGQRQ1
- added IC3: TPS54628DDAR, SOIC127P600X170-9N, symbol TPS54628:TPS54628DDAR
- added IC4: LTC4365ITS8-1#TRPBF, SOT65P280X100-8N, symbol LTC4365ITS8-1#TRPBF:LTC4365ITS8-1#TRPBF
- added J1, J4, J7: Conn_01x04, Connector_PinHeader_2.54mm:PinHeader_1x04_P2.54mm_Vertical, symbol Connector_Generic:Conn_01x04
- added J2, J5: Conn_01x06, Connector_PinHeader_2.54mm:PinHeader_1x06_P2.54mm_Vertical, symbol Connector_Generic:Conn_01x06
- added J3, J6, J8: Conn_01x02, symbol Connector_Generic:Conn_01x02
- added JP1, JP2, JP3, JP4, JP5, JP6, JP7, JP8: Jumper_3_Open, symbol Jumper:Jumper_3_Open
- added L1: 3.3uH, symbol Device:L
- added Q1, Q2: STP130N6F7, TO255P460X1020X2008-3P, symbol STP130N6F7:STP130N6F7
- added R10: 140k, symbol Device:R
- added R11: 160k, symbol Device:R
- added R12, R13, R14, R15, R19, R20, R21: 2.7k, symbol Device:R
- added R16, R8: 100k, symbol Device:R
- added R17: 18k, symbol Device:R
- added R18, R7: 4.7k, symbol Device:R
- added R2, R3, SR_R1, SR_R2: R, symbol Device:R
- added R4, R_IP1, R_IP2: 1k, symbol Device:R
- added R5: 10k, symbol Device:R
- added R9: 4.5M, symbol Device:R
Connections:
- new net: D1.2 (A), R12.2
- new net: IC2.1 (SR/SCLK), JP5.2 (C)
- new net: IC2.2 (DIAG/nSCS), JP6.2 (C)
- new net: IC2.27 (MODE/SDO), JP8.2 (C)
- new net: IC2.28 (ITRIP/SDI), JP7.2 (C)
- new net: D8.2 (A), R21.2
- new net: JP2.3 (B), SR_R1.1
- new net: C10.2, C8.2, C9.2
- new net: D3.2 (A), R14.2
- new net: IC4.2 (UV), R10.1, R9.2
- new net: IC4.3 (OV), R10.2, R11.1
- new net: 5VLED.2 (A), R4.2
- new net: IC3.1 (EN), R5.2
- new net: C11.2, IC3.2 (VFB), R2.2, R3.1
- new net: C4.1, IC3.3 (VREG5)
- new net: C12.1, IC3.4 (SS)
- new net: C5.2, IC3.6 (SW), L1.1
- new net: C5.1, IC3.7 (VBST)
- new net: IC4.5 (~{SHDN}), R8.2
- new net: IC4.8 (GATE), Q1.1 (G), Q2.1 (G)
- new net: D_R2.1, JP5.3 (B)
- new net: C6.2, C7.2, L1.2
- new net: Q1.3 (S), Q2.3 (S)
- new net: D4.2 (A), R15.2
- new net: IC1.28 (ITRIP/SDI), JP3.2 (C)
- new net: JP3.3 (B), R_IT1.2
- new net: JP8.3 (B), R_M2.1
- new net: IC1.1 (SR/SCLK), JP1.2 (C)
- new net: D_R1.1, JP1.3 (B)
- new net: JP7.3 (B), R_IT2.2
- new net: D2.2 (A), R13.2
- new net: JP6.3 (B), SR_R2.1
- new net: IC1.2 (DIAG/nSCS), JP2.2 (C)
- new net: IC1.27 (MODE/SDO), JP4.2 (C)
- new net: D7.2 (A), R20.2
- new net: JP4.3 (B), R_M1.1
- new net: D6.2 (A), R19.2
- new net 12V: C10.1, C17.1, C18.1, C19.1, C21.1, C22.1, C8.1, C9.1, IC1.21 (VM_4), IC1.22 (VM_5), IC1.23 (VM_6), IC1.6 (VM_1), IC1.7 (VM_2), IC1.8 (VM_3), IC2.21 (VM_4), IC2.22 (VM_5), IC2.23 (VM_6), IC2.6 (VM_1), IC2.7 (VM_2), IC2.8 (VM_3), IC3.8 (VIN), IC4.7 (VOUT), Q2.2 (D), R16.1, R19.1
- new net 12V_B: F1.1, J8.1 (Pin_1)
- new net 12V_FUSE: D5.1, F1.2
- new net 12_TVS: IC4.1 (VIN), Q1.2 (D), R8.1, R9.1
- new net 3V3: R18.2, R7.2
- new net 5V: C11.1, J7.1 (Pin_1), R2.1, R4.1
- new net 5V_EN: R5.1
- new net BATTERY_V: J7.4 (Pin_4), R16.2, R17.1
- new net BATTER_FAULT_N: IC4.6 (~{FAULT}), J7.3 (Pin_3)
- new net GND: C16.2, C17.2, C18.2, C19.2, C20.2, C21.2, C22.2, D1.1 (K), D2.1 (K), D3.1 (K), D4.1 (K), D5.2, D6.1 (K), D7.1 (K), D8.1 (K), D_R1.2, D_R2.2, IC1.12 (GND_1), IC1.13 (GND_2), IC1.14 (GND_3), IC1.15 (GND_4), IC1.16 (GND_5), IC1.17 (GND_6), IC1.29 (EP), IC2.12 (GND_1), IC2.13 (GND_2), IC2.14 (GND_3), IC2.15 (GND_4), IC2.16 (GND_5), IC2.17 (GND_6), IC2.29 (EP), IC4.4 (GND), J7.2 (Pin_2), J8.2 (Pin_2), R11.2, R17.2, R_IP1.2, R_IP2.2, R_IT1.1, R_IT2.1, R_M1.2, R_M2.2, SR_R1.2, SR_R2.2
- new net GND2: 5VLED.1 (K), C12.2, R3.2
- new net M1_DRVOFF: IC1.5 (DRVOFF), J2.3 (Pin_3), R20.1
- new net M1_EN/IN1: IC1.4 (EN/IN1)
- new net M1_IPROPI: C16.1, IC1.25 (IPROPI), R_IP1.1
- new net M1_NFAULT: IC1.26 (NFAULT), J2.4 (Pin_4), R7.1
- new net M1_NPROPI: J2.5 (Pin_5)
- new net M1_NSLEEP: IC1.24 (NSLEEP), J2.6 (Pin_6)
- new net M1_OUT1: IC1.10 (OUT1_2), IC1.11 (OUT1_3), IC1.9 (OUT1_1), J3.1 (Pin_1), R12.1
- new net M1_OUT2: IC1.18 (OUT2_1), IC1.19 (OUT2_2), IC1.20 (OUT2_3), J3.2 (Pin_2), R13.1
- new net M1_PH/IN1: J2.2 (Pin_2)
- new net M1_PH/IN2: IC1.3 (PH/IN2), J2.1 (Pin_1)
- new net M1_SCK: J1.1 (Pin_1)
- new net M1_SCLK: JP1.1 (A)
- new net M1_SDI: J1.4 (Pin_4), JP3.1 (A)
- new net M1_SDO: J1.3 (Pin_3), JP4.1 (A), JP8.1 (A)
- new net M1_mSCS: JP2.1 (A), JP6.1 (A)
- new net M1_nSCS: J1.2 (Pin_2)
- new net M2_DRVOFF: IC2.5 (DRVOFF), J5.3 (Pin_3), R21.1
- new net M2_EN/IN1: IC2.4 (EN/IN1)
- new net M2_IPROPI: C20.1, IC2.25 (IPROPI), R_IP2.1
- new net M2_NFAULT: IC2.26 (NFAULT), J5.4 (Pin_4), R18.1
- new net M2_NPROPI2: J5.5 (Pin_5)
- new net M2_NSLEEP: IC2.24 (NSLEEP), J5.6 (Pin_6)
- new net M2_OUT1: IC2.10 (OUT1_2), IC2.11 (OUT1_3), IC2.9 (OUT1_1), J6.1 (Pin_1), R14.1
- new net M2_OUT2: IC2.18 (OUT2_1), IC2.19 (OUT2_2), IC2.20 (OUT2_3), J6.2 (Pin_2), R15.1
- new net M2_PH/EN1: J5.1 (Pin_1), J5.2 (Pin_2)
- new net M2_PH/IN2: IC2.3 (PH/IN2)
- new net M2_SCK: J4.1 (Pin_1)
- new net M2_SCLK: JP5.1 (A)
- new net M2_SDI: J4.4 (Pin_4), JP7.1 (A)
- new net M2_SDO: J4.3 (Pin_3)
- new net M2_nSCS: J4.2 (Pin_2)
- new net PGND: C4.2, C6.1, C7.1, IC3.5 (GND), IC3.9 (PWPD)
Other:
- note added: "18 [V] üzemi fesz; 20-21 [V] vezetési tart"
- note added: "3 output loads must be combined for support loads"
- note added: "3.3*118/18 = 21.6 [V]-ig mérhetek"
- note added: "Always on: if VIN is on it (max 18 [V])"
- note added: "Battery Protection"
- note added: "Battery:"
- note added: "Bulk condenzators"
- note added: "Capacitor to smooth out the transitions most 15k felett vagja: kapcs 20k?)"
- note added: "DRVOFF-> ha fel van huzva akkor van kikapcsolva; akkor vgitanak ha nem engedelyezett"
- note added: "Ezt az MCUhoz"
- note added: "Fogyasztások"
- note added: "Fuse"
- note added: "HW Modes"
- note added: "III.: HW + SPI(S) VARIANT"
- note added: "INKABB az MCU-rol kapcsolajam amit pedig csak USB-rol taplalok?? MOST ALWAYS ON"
- note added: "JST:"
- note added: "MCU-hoz: 100nF-es kapcatior"
- note added: "Motor Enable LEDs"
- note added: "Motor I:"
- note added: "Motor II:"
- note added: "Motor LEDs"
- note added: "Over voltage: OV = 15V R1 = ((V_OS/I_UV)+R3)/OV*0.5 = (300k+4.5M)/15*0.5 =160k R2 = V_OS/I_UV-R1 = 140k"
- note added: "PAD"
- note added: "PCSU:"
- note added: "PCU for the Control Board:"
- note added: "Polarity and Over / Undervoltage Protection"
- note added: "R1+R2 = UV_leak_max/I_leak = 3mV/10nA = 300 kOhm"
- note added: "Ripple nagyság számítás: lásd 13 old; I_ipp ~= 1.33A -> I_max = 5.68A (current rangenek nagyobbnak kell ennel lennie) I_RMS = 5.02 [A] (RMS aramnak nagyobbnak kell lennie)"
- note added: "Standby: the mosfets does not drive the system Activte: the mostfets are currently driving the system Retry: the system trys again after a failure Latch: The system does not try again until the fault is deleted (with nSleep)"
- note added: "Under voltage: UV = 8V -> R3 = U_OS/I_UV*(UV-0.05)/0.5)=300k*(8-0.5)/0.5 = 4.5M"
- note added: "V_out = 0.765(1+R1/R2) R1/R2 ~= 5.534"
- note added: "Voltage Regualtor: I_TRIP = V_ITRIP/R_IPROPI*A_IPROPI"
- note added: "Voltage meas:"
- note added: "Voltage proportional to the current of the motor I_IPROPI = I_motor/4570 V_IPROPI = R*I_IPROPI"
- note added: "Voltage spike protection (TVS)"
- note added: "costum pad-ot csinalni: 5x5mm-es pad; arra kozvetlenul forrasztani a vezekeket"
- note added: "kapcsoló - XT60-as"
- note added: "nem biztos h kell-> csak hosszu vezeteknel kell a vedelem ele erdemes lehet belerakni a nyakba max nem beforrrasztani"
- note added: "tss = 1.15 ms (22-vel: 3.09 ms..)"
- note added: "voltage divider after the battery protection:"

Commit message: Nagyobb lábú MCU implementálás előtt
Parts:
- removed R18, R7: 4.7k, symbol Device:R
Connections:
- net M1_NPROPI is gone; now on net M1_IPROPI: J2.5 (Pin_5)
- net M1_PH/IN1 is gone; now on net M1_EN/IN1: J2.2 (Pin_2)
- net M1_nSCS is gone; now on net ~{M1_SCS}: J1.2 (Pin_2)
- net M2_NPROPI2 is gone; now on net M2_IPROPI: J5.5 (Pin_5)
- net BATTERY_V renamed BAT_V
- net BATTER_FAULT_N renamed ~{BAT_FAIL}
- net M1_NFAULT renamed ~{M1_FAULT}
- net M1_NSLEEP renamed ~{M1_SLEEP}
- net M1_mSCS renamed ~{M1_SCS}
- net ~{M1_SCS}: no longer JP6.1 (A)
- net M2_NFAULT renamed ~{M2_FAULT}
- net M2_NSLEEP renamed ~{M2_SLEEP}
- net M2_nSCS renamed ~{M2_SCS}
- net ~{M2_SCS}: now also JP6.1 (A)
Other:
- note added: "(IPROPI: analog)"
- note added: "(analog)"
- note added: "(felhuzo ellenallas: MCU) NFAULTnak NSLEEPnek"
- note added: "Bulk condensators"
- note removed: "Bulk condenzators"
- note removed: "Ezt az MCUhoz"

Commit message: Schematics nagyjából kész
Parts:
- removed 5VLED: LED, symbol Device:LED
- removed C19: 100uF, symbol Device:C
- removed D_R1, D_R2, R_IT1, R_IT2, R_M1, R_M2: 0, symbol Device:R
- removed JP1, JP2, JP3, JP4, JP5, JP6, JP7, JP8: Jumper_3_Open, symbol Jumper:Jumper_3_Open
- removed R5: 10k, symbol Device:R
- removed SR_R1, SR_R2: R, symbol Device:R
- added C16: 10nF, Capacitor_SMD:C_1206_3216Metric_Pad1.33x1.80mm_HandSolder, symbol Device:C
- added C17: 100uF, Capacitor_THT:CP_Radial_D6.3mm_P2.50mm, symbol Device:C_Polarized
- added D1: 5V_R, LED_SMD:LED_0603_1608Metric_Pad1.05x0.95mm_HandSolder, symbol Device:LED
- added NT1, NT2: NetTie_2, symbol Device:NetTie_2
- added R15, R16: 10, Resistor_SMD:R_0603_1608Metric_Pad0.98x0.95mm_HandSolder, symbol Device:R
- added R17: 5.1k, Resistor_SMD:R_0603_1608Metric_Pad0.98x0.95mm_HandSolder, symbol Device:R
- added R3: 10k, Resistor_SMD:R_0603_1608Metric_Pad0.98x0.95mm_HandSolder, symbol Device:R
- C1: renamed from C17; value 100n -> 100nF; footprint (none) -> Capacitor_SMD:C_0603_1608Metric_Pad1.08x0.95mm_HandSolder; Link (none) -> https://hu.mouser.com/en/ProductDetail/YAGEO/CC0603KRX7R8BB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
- C10: renamed from C5; footprint (none) -> Capacitor_SMD:C_0603_1608Metric_Pad1.08x0.95mm_HandSolder
- C11: renamed from C6; footprint (none) -> Capacitor_SMD:C_1206_3216Metric_Pad1.33x1.80mm_HandSolder; Link (none) -> https://hu.mouser.com/en/ProductDetail/Murata-Electronics/G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
- C12: renamed from C7; footprint (none) -> Capacitor_SMD:C_1206_3216Metric_Pad1.33x1.80mm_HandSolder; Link (none) -> https://hu.mouser.com/en/ProductDetail/Murata-Electronics/G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
- C13: renamed from C21; value 100n -> 100nF; footprint (none) -> Capacitor_SMD:C_0603_1608Metric_Pad1.08x0.95mm_HandSolder; Link (none) -> https://hu.mouser.com/en/ProductDetail/YAGEO/CC0603KRX7R8BB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
- C14: renamed from C22; value 470 -> 470uF
- C15: renamed from C20; value 10n -> 100nF; footprint (none) -> Capacitor_SMD:C_0603_1608Metric_Pad1.08x0.95mm_HandSolder; Link (none) -> https://hu.mouser.com/en/ProductDetail/YAGEO/CC0603KRX7R8BB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
- C3: renamed from C11; value C -> DNP; footprint (none) -> Capacitor_SMD:C_0603_1608Metric_Pad1.08x0.95mm_HandSolder; Link (none) -> https://hu.mouser.com/en/ProductDetail/YAGEO/CC0603KRX7R8BB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
- C4: value 0.1uF -> 1uF; footprint (none) -> Capacitor_SMD:C_0603_1608Metric_Pad1.08x0.95mm_HandSolder
- C5: renamed from C10; footprint (none) -> Capacitor_SMD:C_0805_2012Metric_Pad1.18x1.45mm_HandSolder; Link (none) -> https://hu.mouser.com/en/ProductDetail/Murata-Electronics/G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
- C6: renamed from C12; footprint (none) -> Capacitor_SMD:C_0603_1608Metric_Pad1.08x0.95mm_HandSolder
- C7: renamed from C9; footprint (none) -> Capacitor_SMD:C_0805_2012Metric_Pad1.18x1.45mm_HandSolder
- C8: renamed from C16; value 10n -> 100nF; footprint (none) -> Capacitor_SMD:C_0603_1608Metric_Pad1.08x0.95mm_HandSolder; Link (none) -> https://hu.mouser.com/en/ProductDetail/YAGEO/CC0603KRX7R8BB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
- C9: renamed from C8; footprint (none) -> Capacitor_SMD:C_0603_1608Metric_Pad1.08x0.95mm_HandSolder; Link (none) -> https://hu.mouser.com/en/ProductDetail/YAGEO/CC0603KRX7R8BB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
- D2: renamed from D1; value LED -> M1_OUT1_Y; footprint (none) -> LED_SMD:LED_0603_1608Metric_Pad1.05x0.95mm_HandSolder; Link (none) -> https://eu.mouser.com/en/ProductDetail/Kingbright/APG1608SY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
- D3: renamed from D2; value LED -> M1_OUT2_Y; footprint (none) -> LED_SMD:LED_0603_1608Metric_Pad1.05x0.95mm_HandSolder
- D4: renamed from D3; value LED -> M2_OUT1_Y; footprint (none) -> LED_SMD:LED_0603_1608Metric_Pad1.05x0.95mm_HandSolder
- D5: footprint DIONM7959X262N -> Szakdoga_PowerMan:DIONM7959X262N
- D6: renamed from D4; value LED -> M2_OUT2_Y; footprint (none) -> LED_SMD:LED_0603_1608Metric_Pad1.05x0.95mm_HandSolder
- D7: value LED -> M1_OFF_Y; footprint (none) -> LED_SMD:LED_0603_1608Metric_Pad1.05x0.95mm_HandSolder
- D8: value LED -> M2_OFF_Y; footprint (none) -> LED_SMD:LED_0603_1608Metric_Pad1.05x0.95mm_HandSolder
- D9: renamed from D6; value LED -> BAT_R; footprint (none) -> LED_SMD:LED_0603_1608Metric_Pad1.05x0.95mm_HandSolder
- F1: footprint SF1206HHA3000R2 -> Szakdoga_PowerMan:SF1206HHA3000R2
- IC1: value DRV8244HQDGQRQ1 -> DRV8244SQDGQRQ1; footprint SOP50P490X110-29N -> Szakdoga_PowerMan:SOP50P490X110-29N; Manufacturer_Part_Number DRV8244HQDGQRQ1 -> DRV8244SQDGQRQ1; Mouser Part Number 595-DRV8244HQDGQRQ1 -> 595-DRV8244SQDGQRQ1; Mouser Price/Stock https://www.mouser.co.uk/ProductDetail/Texas-Instruments/DR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 -> https://hu.mouser.com/en/ProductDetail/Texas-Instruments/DR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
- IC2: renamed from IC3; footprint SOIC127P600X170-9N -> Szakdoga_PowerMan:SOIC127P600X170-9N
- IC3: renamed from IC2; value DRV8244HQDGQRQ1 -> DRV8244SQDGQRQ1; footprint SOP50P490X110-29N -> Szakdoga_PowerMan:SOP50P490X110-29N; Manufacturer_Part_Number DRV8244HQDGQRQ1 -> DRV8244SQDGQRQ1; Mouser Part Number 595-DRV8244HQDGQRQ1 -> 595-DRV8244SQDGQRQ1; Mouser Price/Stock https://www.mouser.co.uk/ProductDetail/Texas-Instruments/DR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 -> https://hu.mouser.com/en/ProductDetail/Texas-Instruments/DR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
- IC4: footprint SOT65P280X100-8N -> Szakdoga_PowerMan:SOT65P280X100-8N
- J1: renamed from J3; value Conn_01x02 -> MOTOR1_OUT; footprint (none) -> CustomFootprints:Motor_SolderPad_2Pin
- J2: renamed from J1; value Conn_01x04 -> M1_SPI; footprint Connector_PinHeader_2.54mm:PinHeader_1x04_P2.54mm_Vertical -> Connector_JST:JST_XH_S4B-XH-A-1_1x04_P2.50mm_Horizontal
- J3: renamed from J2; value Conn_01x06 -> M1_CTRL; footprint Connector_PinHeader_2.54mm:PinHeader_1x06_P2.54mm_Vertical -> Connector_JST:JST_XH_S6B-XH-A-1_1x06_P2.50mm_Horizontal
- J4: renamed from J6; value Conn_01x02 -> MOTOR2_OUT; footprint (none) -> CustomFootprints:Motor_SolderPad_2Pin
- J5: renamed from J4; value Conn_01x04 -> M2_SPI; footprint Connector_PinHeader_2.54mm:PinHeader_1x04_P2.54mm_Vertical -> Connector_JST:JST_XH_S4B-XH-A-1_1x04_P2.50mm_Horizontal
- J6: renamed from J5; value Conn_01x06 -> M2_CTRL; footprint Connector_PinHeader_2.54mm:PinHeader_1x06_P2.54mm_Vertical -> Connector_JST:JST_XH_S6B-XH-A-1_1x06_P2.50mm_Horizontal
- J7: value Conn_01x04 -> 5V_CON; footprint Connector_PinHeader_2.54mm:PinHeader_1x04_P2.54mm_Vertical -> Connector_JST:JST_XH_S4B-XH-A-1_1x04_P2.50mm_Horizontal
- J8: value Conn_01x02 -> BAT_CON; footprint (none) -> CustomFootprints:Battery_SolderPad_2Pin
- L1: footprint (none) -> Szakdoga_PowerMan:BMRA000606303R3MA1; Link (none) -> https://hu.mouser.com/en/ProductDetail/Pulse-Electronics/BM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
- Q1, Q2: footprint TO255P460X1020X2008-3P -> Szakdoga_PowerMan:TO255P460X1020X2008-3P
- R1: renamed from R2; value R -> 124k; footprint (none) -> Resistor_SMD:R_0603_1608Metric_Pad0.98x0.95mm_HandSolder
- R10: renamed from R21; value 2.7k -> 1k; footprint (none) -> Resistor_SMD:R_0603_1608Metric_Pad0.98x0.95mm_HandSolder
- R11: renamed from R9; footprint (none) -> Resistor_SMD:R_0603_1608Metric_Pad0.98x0.95mm_HandSolder
- R12: renamed from R10; footprint (none) -> Resistor_SMD:R_0603_1608Metric_Pad0.98x0.95mm_HandSolder
- R13: renamed from R11; footprint (none) -> Resistor_SMD:R_0603_1608Metric_Pad0.98x0.95mm_HandSolder
- R14: renamed from R8; footprint (none) -> Resistor_SMD:R_0603_1608Metric_Pad0.98x0.95mm_HandSolder
- R18: renamed from R19; footprint (none) -> Resistor_SMD:R_0603_1608Metric_Pad0.98x0.95mm_HandSolder
- R19: renamed from R16; footprint (none) -> Resistor_SMD:R_0603_1608Metric_Pad0.98x0.95mm_HandSolder
- R2: renamed from R3; value R -> 22.1k; footprint (none) -> Resistor_SMD:R_0603_1608Metric_Pad0.98x0.95mm_HandSolder
- R20: renamed from R17; footprint (none) -> Resistor_SMD:R_0603_1608Metric_Pad0.98x0.95mm_HandSolder
- R4, R_IP1, R_IP2: footprint (none) -> Resistor_SMD:R_0603_1608Metric_Pad0.98x0.95mm_HandSolder
- R5: renamed from R12; footprint (none) -> Resistor_SMD:R_0603_1608Metric_Pad0.98x0.95mm_HandSolder
- R6: renamed from R13; footprint (none) -> Resistor_SMD:R_0603_1608Metric_Pad0.98x0.95mm_HandSolder
- R7: renamed from R14; footprint (none) -> Resistor_SMD:R_0603_1608Metric_Pad0.98x0.95mm_HandSolder
- R8: renamed from R15; footprint (none) -> Resistor_SMD:R_0603_1608Metric_Pad0.98x0.95mm_HandSolder
- R9: renamed from R20; value 2.7k -> 1k; footprint (none) -> Resistor_SMD:R_0603_1608Metric_Pad0.98x0.95mm_HandSolder
- renumbered C18 to C2
Connections:
- net GND2 is gone; now on net GND: C6.2, R2.2
- net M1_SCK is gone; now on net M1_SCLK: J2.1 (Pin_1)
- net M2_SCK is gone; now on net M2_SCLK: J5.1 (Pin_1)
- net PGND is gone; now on net GNDPWR: C11.1, C12.1, C4.2, IC2.5 (GND), IC2.9 (PWPD)
- net 12V: now also C17.1, R3.2
- net 12V_FUSE: now also NT1.1; no longer D5.1
- net 5V: now also C11.2, C12.2, L1.2
- net GND: now also D1.1 (K), NT2.2; no longer C1.2, C13.2, C14.2, C15.2, C2.2, C8.2, D2.1 (K), D3.1 (K), D4.1 (K), D5.2, D6.1 (K), D9.1 (K), IC1.12 (GND_1), IC1.13 (GND_2), IC1.14 (GND_3), IC1.15 (GND_4), IC1.16 (GND_5), IC1.17 (GND_6), IC1.29 (EP), IC3.12 (GND_1), IC3.13 (GND_2), IC3.14 (GND_3), IC3.15 (GND_4), IC3.16 (GND_5), IC3.17 (GND_6), IC3.29 (EP), J8.2 (Pin_2), R20.2, R_IP1.2, R_IP2.2
- net M1_SCLK: now also IC1.1 (SR/SCLK)
- net M1_SDI: now also IC1.28 (ITRIP/SDI)
- net M1_SDO: now also IC1.27 (MODE/SDO)
- net M2_EN/IN1: now also J6.2 (Pin_2)
- net M2_PH/IN2: now also J6.1 (Pin_1)
- net M2_SCLK: now also IC3.1 (SR/SCLK)
- net M2_SDI: now also IC3.28 (ITRIP/SDI)
- net M2_SDO: now also IC3.27 (MODE/SDO)
- net ~{M1_SCS}: now also IC1.2 (DIAG/nSCS)
- net ~{M2_SCS}: now also IC3.2 (DIAG/nSCS)
- net GNDPWR: now reaches C5.2, C7.2, C9.2
- net GNDPWR: now also C1.2, C13.2, C14.2, C15.2, C2.2, C8.2, D2.1 (K), D3.1 (K), D4.1 (K), D5.2, D6.1 (K), D9.1 (K), IC1.12 (GND_1), IC1.13 (GND_2), IC1.14 (GND_3), IC1.15 (GND_4), IC1.16 (GND_5), IC1.17 (GND_6), IC1.29 (EP), IC3.12 (GND_1), IC3.13 (GND_2), IC3.14 (GND_3), IC3.15 (GND_4), IC3.16 (GND_5), IC3.17 (GND_6), IC3.29 (EP), J8.2 (Pin_2), R20.2, R_IP1.2, R_IP2.2, C16.2, C17.2, NT2.1
- net at R4.2: now also D1.2 (A)
- net at IC2.1 (EN): now also R3.1
- removed net M2_PH/EN1: J6.1 (Pin_1), J6.2 (Pin_2)
- new net: IC4.8 (GATE), R15.1, R16.2, R17.2
- new net: C16.1, R17.1
- new net: Q1.1 (G), R15.2
- new net: Q2.1 (G), R16.1
- new net 12V_TVS: D5.1, NT1.2
Other:
- note added: "1% >"
- note added: "16 VDC"
- note added: "25 VDC"
- note added: "CSAK SPI verzio maradt"
- note added: "Inrush prot"
- note added: "Motor Driver OFF LEDs"
- note added: "SPI (S) variant Motor Controls:"
- note added: "Vout = 0.765*(1+R1/R2) = 5.05 [V]"
- note added: "behuzni h folyton fennlegyen"
- note added: "esetleg ide egy kis keramia kondi?"
- note removed: "III.: HW + SPI(S) VARIANT"
- note removed: "Motor Enable LEDs"
- moved on the sheet: C3, D3, D5, D6, D7, D8, Q1, R1, R18, R8, R_IP2
